File: HackFFM-Duino Chime.sch (EAGLE design)
At the start: 63 parts, among them IC1 ATMEGA328, IC2 SN74LVC2G14, IC3 74LVC1G53DP, Q1 16MHz, U2 3.3V MIC5205, U3 MAX98306ETD+, U4 3.3V MIC5205

Commit message: Version 1.1 update
Parts:
- removed D8: M01M01_SMDSHORT_NOCREAM, MyEagleLibrary:M01M01_SMDSHORT_NOCREAM
- removed MONO_R0: 0R, MyEagleLibrary:R-EU_R0805
- removed U$1: MICROSD, MyEagleLibrary:MICROSD
- added A2: M01M01_SMD_EDGE_SHORT, MyEagleLibrary:M01M01_SMD_EDGE_SHORT
- added SJ1: SOLDERJUMPERNO, SparkFun:SOLDERJUMPERNO
- added XU1: MICROSD_DETMOLEX104031, DCEM-microSD:MICROSD_DETMOLEX104031
- +5V, 1+, 1-, 2+, 2-, A0, A4, A5, D3, D5, D6, D7, GND: value M01M01_SMDSHORT_NOCREAM -> M01M01_SMD_EDGE_SHORT; device MyEagleLibrary:M01M01_SMDSHORT_NOCREAM -> MyEagleLibrary:M01M01_SMD_EDGE_SHORT
- CTS, DTR, GND_, MISO, MOSI, RST, RXI, SCK, TXO, VCC: value M01M01_SMDSHORT_NOCREAM -> M01M01_SMD_EDGE_XS; device MyEagleLibrary:M01M01_SMDSHORT_NOCREAM -> MyEagleLibrary:M01M01_SMD_EDGE_XS
Connections:
- removed net 3.3V: C1.1, C10.1, C3.2, IC1.AVCC, IC1.VCC@1, IC1.VCC@2, R2.2, R5.2, R7.2, U$1.VDD, U2.OUT, VCC.1
- new net +3V3: C1.1, C10.1, C3.2, IC1.AVCC, IC1.VCC@1, IC1.VCC@2, R2.2, R5.2, R7.2, U2.OUT, VCC.1
- net A2: now also A2.1; no longer U$1.CARD_DETECT
- net D4: now also XU1G$1.!CS; no longer U$1.CS
- net D8: now also XU1G$1.DET_A; no longer D8.1
- net GND: no longer U$1.CARD_DETECT1, U$1.GND, U$1.GND1, U$1.VSS
- net MISO: now also XU1G$1.MISO; no longer U$1.DATA_OUT
- net MOSI: now also XU1G$1.MOSI; no longer U$1.DATA_IN
- net N$15: now also SJ1.1; no longer MONO_R0.1
- net N$17: now also SJ1.2; no longer MONO_R0.2
- net SCK: now also XU1G$1.SCK; no longer U$1.SCLK
Other:
- note added: "O: stereo C: mono"
- note added: "Version 1.1"
- note removed: "Version 1.0"
